Commit message: amr_mini

File: urdf/urdf_include/lidar.xacro (robot description, xacro)
@@ -15,5 +15,5 @@
                 <mesh filename="file://$(find amr_mini_description)/AmrMini_models/Amr_mini/meshes/lidar.stl" scale="0.001 0.001 0.001"/>
               </geometry>
-              <origin rpy="${pi} 0 -${pi/1.3}" xyz="-0.075 0 0"/>
+              <origin rpy="${pi} 0 -${pi/1.25}" xyz="-0.075 0.02 0"/>
             </visual>
             <collision>
@@ -21,5 +21,5 @@
                 <mesh filename="file://$(find amr_mini_description)/AmrMini_models/Amr_mini/meshes/lidar.stl" scale="0.001 0.001 0.001"/>
               </geometry>
-              <origin rpy="${pi} 0 -${pi/1.3}" xyz="-0.075 0 0"/>
+              <origin rpy="${pi} 0 -${pi/1.25}" xyz="-0.078 0 0"/>
             </collision>
             <inertial>
@@ -37,5 +37,5 @@
           <always_on>true</always_on>
           <visualize>true</visualize>
-          <update_rate>10</update_rate>
+          <update_rate>2</update_rate>
           <ray>
             <scan>
@@ -43,6 +43,6 @@
                 <samples>270</samples>
                 <resolution>1.00000</resolution>
-                <min_angle>-1.45</min_angle>
-                <max_angle>2.36</max_angle>
+                <min_angle>-1.45245</min_angle>
+                <max_angle>2.7159</max_angle>
               </horizontal>
             </scan>
