Commit message: Amr_mini

File: urdf/amr_mini_xacro.urdf (robot description, URDF)
Before this commit: robot AmrRobot, 18 links, 17 joints
Links:
- link back_left_caster_rotation_link: geometry collision mesh filename=file:///home/mkutan/Documents/ros2_ws/install/amr_mini_desc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 scale=1 1 0.9; visual mesh filename=file:///home/mkutan/Documents/ros2_ws/install/amr_mini_desc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 scale=1 1 0.9
- link back_lidar_laser_link: geometry collision mesh filename=file:///home/mkutan/Documents/ros2_ws/install/amr_mini_desc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 scale=0.001 0.001 0.001; visual mesh filename=file:///home/mkutan/Documents/ros2_ws/install/amr_mini_desc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 scale=0.001 0.001 0.001
- link back_right_caster_rotation_link: geometry collision mesh filename=file:///home/mkutan/Documents/ros2_ws/install/amr_mini_desc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 scale=1 1 0.9; visual mesh filename=file:///home/mkutan/Documents/ros2_ws/install/amr_mini_desc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 scale=1 1 0.9
- link base_link: geometry collision mesh filename=file:///home/mkutan/Documents/ros2_ws/install/amr_mini_desc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 scale=0.001 0.001 0.001; visual mesh filename=file:///home/mkutan/Documents/ros2_ws/install/amr_mini_desc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 scale=0.001 0.001 0.001
- link camera: geometry collision mesh filename=file:///home/mkutan/Documents/ros2_ws/install/amr_mini_desc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; visual mesh filename=file:///home/mkutan/Documents/ros2_ws/install/amr_mini_desc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
- link front_left_caster_rotation_link: geometry collision mesh filename=file:///home/mkutan/Documents/ros2_ws/install/amr_mini_desc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 scale=1 1 0.9; visual mesh filename=file:///home/mkutan/Documents/ros2_ws/install/amr_mini_desc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 scale=1 1 0.9
- link front_lidar_laser_link: geometry collision mesh filename=file:///home/mkutan/Documents/ros2_ws/install/amr_mini_desc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 scale=0.001 0.001 0.001; visual mesh filename=file:///home/mkutan/Documents/ros2_ws/install/amr_mini_desc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 scale=0.001 0.001 0.001
- link front_right_caster_rotation_link: geometry collision mesh filename=file:///home/mkutan/Documents/ros2_ws/install/amr_mini_desc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 scale=1 1 0.9; visual mesh filename=file:///home/mkutan/Documents/ros2_ws/install/amr_mini_desc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 scale=1 1 0.9
- link imu: geometry collision mesh filename=file:///home/mkutan/Documents/ros2_ws/install/amr_mini_desc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 scale=0.001 0.001 0.001; visual mesh filename=file:///home/mkutan/Documents/ros2_ws/install/amr_mini_desc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 scale=0.001 0.001 0.001
- link left_motor: geometry collision mesh filename=file:///home/mkutan/Documents/ros2_ws/install/amr_mini_desc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 scale=0.001 0.001 0.00065; visual mesh filename=file:///home/mkutan/Documents/ros2_ws/install/amr_mini_desc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 scale=0.001 0.001 0.00065
- link left_wheel: geometry collision mesh filename=file:///home/mkutan/Documents/ros2_ws/install/amr_mini_desc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 scale=0.001 0.001 0.001; visual mesh filename=file:///home/mkutan/Documents/ros2_ws/install/amr_mini_desc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 scale=0.001 0.001 0.001
- link right_motor: geometry collision mesh filename=file:///home/mkutan/Documents/ros2_ws/install/amr_mini_desc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 scale=0.001 0.001 0.00065; visual mesh filename=file:///home/mkutan/Documents/ros2_ws/install/amr_mini_desc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 scale=0.001 0.001 0.00065
- link right_wheel: geometry collision mesh filename=file:///home/mkutan/Documents/ros2_ws/install/amr_mini_desc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 scale=0.001 0.001 0.001; visual mesh filename=file:///home/mkutan/Documents/ros2_ws/install/amr_mini_desc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 scale=0.001 0.001 0.001
