Commit message: amr_mini

File: urdf/amr_mini.xacro (robot description, xacro)
@@ -49,5 +49,5 @@
     <!-- Left Lidar-->
     <xacro:lidar name="front_lidar" parent="base_link">
-      <origin rpy="${pi} 0 -2.30 " xyz="-${lidar_x} -${lidar_y} ${lidar_z}"/>
+      <origin rpy="${pi} 0 -2.34" xyz="-${lidar_x} -${lidar_y} ${lidar_z}"/>
     </xacro:lidar>
     <!--imu-->

File: urdf/urdf_include/base_link.xacro (robot description, xacro)
@@ -28,8 +28,8 @@
           </inertial>
       </link>
-      <!-- <gazebo reference="${name}">
+      <gazebo reference="${name}">
         <material>
           Gazebo/Turquoise</material>
-      </gazebo> -->
+      </gazebo>
   </xacro:macro>
 </robot>

File: urdf/urdf_include/camera.xacro (robot description, xacro)
@@ -25,17 +25,9 @@
                 o_xyz="0 0 0" o_rpy="0 0 0" />
         </link>
-       <!-- <gazebo reference="${name}">
+       <gazebo reference="${name}">
         <sensor type="depth" name="depth_camera">
             <visualize>true</visualize>
             <update_rate>10.0</update_rate>
             <plugin name="${name}_depth_plugin" filename="libgazebo_ros_camera.so">
-              <!-
-               Change namespace, camera name and topics so -
-                   * Raw images are published to: /custom_ns/custom_camera/custom_image
-                   * Depth images are published to: /custom_ns/custom_camera/custom_image_depth
-                   * Raw image camera info is published to: /custom_ns/custom_camera/custom_info_raw
-                   * Depth image camera info is published to: /custom_ns/custom_camera/custom_info_depth
-                   * Point cloud is published to: /custom_ns/custom_camera/custom_points
-              ->
               <ros>
                 <namespace>amr_mini_description</namespace>
@@ -44,11 +36,11 @@
                 <remapping>custom_camera/camera_info:=custom_camera/custom_info_raw</remapping>
                 <remapping>custom_camera/camera_info_depth:=custom_camera/custom_info_depth</remapping>
-                <remapping>custom_camera/points:=custom_camera/custom_points</remapping>  <!-#pointCloudTopicName->
+                <remapping>custom_camera/points:=custom_camera/custom_points</remapping>
               </ros>
             <camera_name>custom_camera</camera_name>
               <frame_name>${name}</frame_name>
               <hack_baseline>0.07</hack_baseline>
-               <min_depth>0.001</min_depth> <!-#pointCloudCutoff ->
-               <max_depth>300.0</max_depth> <!-#pointCloudCutoffMax ->
+               <min_depth>0.001</min_depth>
+               <max_depth>300.0</max_depth>
             </plugin>
             </sensor>
@@ -69,5 +61,5 @@
             </plugin>
         </sensor>
-        </gazebo> -->
+        </gazebo>
     </xacro:macro>
 </robot>

File: urdf/urdf_include/caster_wheel.xacro (robot description, xacro)
@@ -39,8 +39,8 @@
           <xacro:default_inertial mass="0.21"/>
       </link>
-      <!-- <gazebo reference="${locationprefix}_caster_rotation_link">
+      <gazebo reference="${locationprefix}_caster_rotation_link">
         <material>
           Gazebo/Orange</material>
-    </gazebo> -->
+    </gazebo>
       <xacro:caster_wheel_link parent="${locationprefix}_caster_rotation_link" locationprefix="${locationprefix}">
         <origin rpy="${pi*0.5} 0 0 " xyz="${amr_mini_caster_wheel_dx} ${-amr_mini_caster_wheel_dy * locationright} ${amr_mini_caster_wheel_dz*8.8}"/>

File: urdf/urdf_include/caster_wheel_link.xacro (robot description, xacro)
@@ -31,5 +31,5 @@
           o_xyz="0 0 0" o_rpy="0 0 0" />
       </link>
-      <!-- <gazebo reference="${locationprefix}_caster_wheel_link">
+      <gazebo reference="${locationprefix}_caster_wheel_link">
         <material>Gazebo/Red</material>
       </gazebo>
@@ -43,5 +43,5 @@
         <minDepth>0.001</minDepth>
         <maxVel>1.0</maxVel>
-      </gazebo> -->
+      </gazebo>
   </xacro:macro>
 </robot>

File: urdf/urdf_include/gazebo.xacro (robot description, xacro)
@@ -3,39 +3,40 @@
   <xacro:macro name="gazebo_diff">
     <gazebo>
-        <plugin name='diff_drive' filename='libgazebo_ros_diff_drive.so'>
-          <ros>
-            <namespace>amr_mini_description</namespace>
-          </ros>
-          <update_rate>30</update_rate>
-          <left_joint>left_wheel_joint</left_joint>
-          <right_joint>right_wheel_joint</right_joint>
-          <wheel_separation>0.464</wheel_separation>
-          <wheel_diameter>0.2</wheel_diameter>
-          <wheel_separation>0.160</wheel_separation>
-          <max_wheel_acceleration>0.07</max_wheel_acceleration>
-          <command_topic>cmd_vel</command_topic>
-          <publish_odom>true</publish_odom>
-          <publish_odom_tf>true</publish_odom_tf>
-          <publish_wheel_tf>false</publish_wheel_tf>
-          <odometry_topic>odom</odometry_topic>
-          <odometry_frame>odom</odometry_frame>
-          <robot_base_frame>base_footprint</robot_base_frame>
-        </plugin>
-        <plugin name="basic_joint_state" filename="libgazebo_ros_joint_state_publisher.so">
-          <ros>
-            <remapping>~/out:=joint_states</remapping>
-          </ros>
-          <update_rate>30</update_rate>
-          <joint_name>left_wheel_joint</joint_name>
-          <joint_name>right_wheel_joint</joint_name>
-          <joint_name>back_left_caster_wheel_joint</joint_name>
-          <joint_name>back_right_caster_wheel_joint</joint_name>
-          <joint_name>front_right_caster_wheel_joint</joint_name>
-          <joint_name>front_left_caster_wheel_joint</joint_name>
-          <joint_name>back_left_caster_rotation_joint</joint_name>
-          <joint_name>back_right_caster_rotation_joint</joint_name>
-          <joint_name>front_right_caster_rotation_joint</joint_name>
-          <joint_name>front_left_caster_rotation_joint</joint_name>
-        </plugin>
+      <plugin name='diff_drive' filename='libgazebo_ros_diff_drive.so'>
+        <ros>
+          <namespace>amr_mini_description</namespace>
+        </ros>
+        <update_rate>30</update_rate>
+        <left_joint>left_wheel_joint</left_joint>
+        <right_joint>right_wheel_joint</right_joint>
+        <wheel_diameter>0.08</wheel_diameter>
+        <wheel_separation>0.21</wheel_separation>
+        <max_wheel_torque>20</max_wheel_torque>
+        <max_wheel_acceleration>10</max_wheel_acceleration>
+        <command_topic>cmd_vel</command_topic>
+        <cmd_vel_timeout>0.5</cmd_vel_timeout>
+        <publish_odom>true</publish_odom>
+        <publish_odom_tf>false</publish_odom_tf>
+        <publish_wheel_tf>false</publish_wheel_tf>
+        <odometry_topic>odom</odometry_topic>
+        <odometry_frame>odom</odometry_frame>
+        <robot_base_frame>base_footprint</robot_base_frame>
+      </plugin>
+      <plugin name='basic_joint_state' filename='libgazebo_ros_joint_state_publisher.so'>
+        <ros>
+          <remapping>~/out:=joint_states</remapping>
+        </ros>
+        <update_rate>30</update_rate>
+        <joint_name>left_wheel_joint</joint_name>
+        <joint_name>right_wheel_joint</joint_name>
+        <joint_name>back_left_caster_wheel_joint</joint_name>
+        <joint_name>back_right_caster_wheel_joint</joint_name>
+        <joint_name>front_right_caster_wheel_joint</joint_name>
+        <joint_name>front_left_caster_wheel_joint</joint_name>
+        <joint_name>back_left_caster_rotation_joint</joint_name>
+        <joint_name>back_right_caster_rotation_joint</joint_name>
+        <joint_name>front_right_caster_rotation_joint</joint_name>
+        <joint_name>front_left_caster_rotation_joint</joint_name>
+      </plugin>
       </gazebo>
   </xacro:macro>

File: urdf/urdf_include/imu.xacro (robot description, xacro)
@@ -21,5 +21,5 @@
             </collision>
         </link>
-        <!-- <gazebo reference="${name}">
+       <gazebo reference="${name}">
             <material>Gazebo/Yellow</material>
         </gazebo>
@@ -37,5 +37,5 @@
             </plugin>
           </sensor>
-        </gazebo> -->
+        </gazebo>
     </xacro:macro>
 </robot>

File: urdf/urdf_include/lidar.xacro (robot description, xacro)
@@ -1,9 +1,9 @@
 <?xml version="1.0"?>
-<robot xmlns:xacro="http://www.ros.org/wiki/xacro" name="ArmRobot">
+<robot xmlns:xacro="http://www.ros.org/wiki/xacro" name="AmrRobot">
 <xacro:property name="pi" value="3.14"/>
 <!-- inertial-->
 <xacro:include filename="$(find amr_mini_description)/urdf/urdf_include/common_properties.urdf.xacro"/>
   <xacro:macro name="lidar" params="name parent *origin">
-      <joint name="${name}_joint" type="fixed">
+      <joint name="${name}_joint" type="continuous">
           <xacro:insert_block name="origin"/>
           <parent link="${parent}"/>
@@ -21,8 +21,13 @@
                 <mesh filename="file://$(find amr_mini_description)/AmrMini_models/Amr_mini/meshes/lidar.stl" scale="0.001 0.001 0.001"/>
               </geometry>
-              <origin rpy="0 0 ${pi}" xyz="-0.072 -0.085 0.02"/>
+              <origin rpy="${pi} 0 ${pi}" xyz="-0.072 -0.085 0.02"/>
             </collision>
+            <inertial>
+              <origin xyz="0 0 0" rpy="0 0 0" />
+              <mass value="1.5" />
+              <inertia ixx="0.0075" ixy="0.0" ixz="0.0" iyy="0.0085" iyz="0.0" izz="0.0085" />
+            </inertial>
       </link>
-    <!-- <gazebo reference="${name}_laser_link">
+  <gazebo reference="${name}_laser_link">
         <material>Gazebo/Yellow</material>
     </gazebo>
@@ -31,5 +36,5 @@
           <pose>0 0 0 0 0 0</pose>
           <visualize>true</visualize>
-          <update_rate>15</update_rate>
+          <update_rate>5</update_rate>
           <ray>
             <scan>
@@ -37,11 +42,11 @@
                 <samples>270</samples>
                 <resolution>1</resolution>
-                <min_angle>-1.45245</min_angle>
-                <max_angle>2.34159</max_angle>
+                <min_angle>-1.0</min_angle>
+                <max_angle>2.0</max_angle>
               </horizontal>
             </scan>
             <range>
               <min>0.10</min>
-              <max>30.0</max>
+              <max>15</max>
               <resolution>0.01</resolution>
             </range>
@@ -54,5 +59,4 @@
           <plugin name="gazebo_ros_head_hokuyo_controller" filename="libgazebo_ros_ray_sensor.so">
             <ros>
-              <namespace>amr_mini_description</namespace>
               <remapping>~/out:=${name}_amr_mini_laser</remapping>
             </ros>
@@ -61,5 +65,5 @@
           </plugin>
         </sensor>
-      </gazebo>   -->
+      </gazebo>
   </xacro:macro>
 </robot>

File: urdf/urdf_include/motor.xacro (robot description, xacro)
@@ -23,8 +23,8 @@
           </collision>
       </link>
-         <!-- <gazebo reference="${name}">
+         <gazebo reference="${name}">
       <material>
         Gazebo/Blue</material>
-  </gazebo> -->
+  </gazebo>
   </xacro:macro>
 </robot>

File: urdf/urdf_include/wheel.xacro (robot description, xacro)
@@ -33,5 +33,5 @@
             </inertial>
         </link>
-        <!-- <gazebo reference="${name}_wheel">
+        <gazebo reference="${name}_wheel">
           <material>
             Gazebo/Trunk</material>
@@ -45,5 +45,6 @@
             <maxVel>1.0</maxVel>
         </gazebo> -->
-          <!-- <ros2_control name="GazeboSystem" type="system">
+<!--
+          <ros2_control name="GazeboSystem" type="system">
             <hardware>
               <plugin>gazebo_ros2_control/GazeboSystem</plugin>

Commit message: amr_mini

File: urdf/amr_mini.xacro (robot description, xacro)
@@ -6,7 +6,7 @@
     <xacro:property name="wheel_y" value="0.25"/>
     <xacro:property name="wheel_z" value="0.002"/>
-    <xacro:property name="lidar_z" value="0.21"/>
-    <xacro:property name="lidar_x" value="0.37"/>
-    <xacro:property name="lidar_y" value="0.223"/>
+    <xacro:property name="lidar_z" value="0.19"/>
+    <xacro:property name="lidar_x" value="0.34"/>
+    <xacro:property name="lidar_y" value="0.220"/>
     <xacro:property name="amr_mini_caster_wheel_radius" value="0.0525" />
     <xacro:property name="amr_mini_caster_wheel_dz" value="0.0112" />
@@ -43,12 +43,16 @@
       <origin rpy="0 0 ${pi}" xyz="${wheel_x} -${wheel_y} ${wheel_z}"/>
     </xacro:wheel>
-    <!-- Right Lidar-->
+    <!-- Back Lidar-->
     <xacro:lidar name="back_lidar" parent="base_link">
-      <origin rpy="${pi} 0 0.78 " xyz="${lidar_x} ${lidar_y} ${lidar_z}"/>
+      <origin rpy="0 0 ${pi/20} " xyz="${lidar_x} ${lidar_y} ${lidar_z}"/>
     </xacro:lidar>
     <!-- Left Lidar-->
     <xacro:lidar name="front_lidar" parent="base_link">
-      <origin rpy="${pi} 0 -2.34" xyz="-${lidar_x} -${lidar_y} ${lidar_z}"/>
+      <origin rpy="0 0 -${pi}" xyz="-${lidar_x} -${lidar_y} ${lidar_z}"/>
     </xacro:lidar>
+    <!-- Lidar-->
+    <!-- <xacro:lidar name="main_lidar" parent="base_link">
+      <origin rpy="${pi} 0 0" xyz="0 0  ${lidar_z+0.165}"/>
+    </xacro:lidar> -->
     <!--imu-->
     <xacro:imu name="imu" parent="base_link">

File: urdf/amr_mini_xacro.urdf (robot description, URDF)
Before this commit: robot AmrRobot, 18 links, 17 joints
Links:
- link back_lidar_laser_link: mass 1.5 -> 0.14
- link front_lidar_laser_link: mass 1.5 -> 0.14
Joints:
- joint back_lidar_joint: origin xyz=0.37 0.223 0.21 rpy=3.141592653589793 0 0.78  -> xyz=0.34 0.22 0.19 rpy=0 0 0.15707963267948966 
- joint front_lidar_joint: origin xyz=-0.37 -0.223 0.21 rpy=3.141592653589793 0 -2.34 -> xyz=-0.34 -0.22 0.19 rpy=0 0 -3.141592653589793

File: urdf/urdf_include/lidar.xacro (robot description, xacro)
@@ -15,5 +15,5 @@
                 <mesh filename="file://$(find amr_mini_description)/AmrMini_models/Amr_mini/meshes/lidar.stl" scale="0.001 0.001 0.001"/>
               </geometry>
-              <origin rpy="0 0 ${pi}" xyz="-0.072 -0.085 0.02"/>
+              <origin rpy="${pi} 0 -${pi/1.3}" xyz="-0.075 0 0"/>
             </visual>
             <collision>
@@ -21,9 +21,9 @@
                 <mesh filename="file://$(find amr_mini_description)/AmrMini_models/Amr_mini/meshes/lidar.stl" scale="0.001 0.001 0.001"/>
               </geometry>
-              <origin rpy="${pi} 0 ${pi}" xyz="-0.072 -0.085 0.02"/>
+              <origin rpy="${pi} 0 -${pi/1.3}" xyz="-0.075 0 0"/>
             </collision>
             <inertial>
               <origin xyz="0 0 0" rpy="0 0 0" />
-              <mass value="1.5" />
+              <mass value="0.14" />
               <inertia ixx="0.0075" ixy="0.0" ixz="0.0" iyy="0.0085" iyz="0.0" izz="0.0085" />
             </inertial>
@@ -35,19 +35,20 @@
       <sensor type="ray" name="${name}_rplidar_sensor">
           <pose>0 0 0 0 0 0</pose>
+          <always_on>true</always_on>
           <visualize>true</visualize>
-          <update_rate>5</update_rate>
+          <update_rate>10</update_rate>
           <ray>
             <scan>
               <horizontal>
                 <samples>270</samples>
-                <resolution>1</resolution>
-                <min_angle>-1.0</min_angle>
-                <max_angle>2.0</max_angle>
+                <resolution>1.00000</resolution>
+                <min_angle>-1.45</min_angle>
+                <max_angle>2.36</max_angle>
               </horizontal>
             </scan>
             <range>
-              <min>0.10</min>
-              <max>15</max>
-              <resolution>0.01</resolution>
+              <min>0.120000</min>
+              <max>20</max>
+              <resolution>0.015000</resolution>
             </range>
             <noise>
