Commit message: Amr_mini

File: urdf/amr_mini.xacro (robot description, xacro)
@@ -14,4 +14,5 @@
     <xacro:property name="amr_mini_front_caster_wheel_base_dz" value="0.0536"/>
     <xacro:property name="locationright" value="1"/>
+   <xacro:arg name="use_nominal_extrinsics" default="false"/>
     <!-- include-->
   <xacro:include filename="$(find amr_mini_description)/urdf/urdf_include/base_link.xacro"/>
@@ -21,6 +22,7 @@
   <xacro:include filename="$(find amr_mini_description)/urdf/urdf_include/caster_wheel.xacro"/>
   <xacro:include filename="$(find amr_mini_description)/urdf/urdf_include/imu.xacro"/>
-  <xacro:include filename="$(find amr_mini_description)/urdf/urdf_include/camera.xacro"/>
   <xacro:include filename="$(find amr_mini_description)/urdf/urdf_include/gazebo.xacro"/>
+  <xacro:include filename="$(find amr_mini_description)/urdf/urdf_include/_d435i.urdf.xacro" />
+  <xacro:include filename="$(find amr_mini_description)/urdf/urdf_include/intel_d435.urdf.xacro" />
     <!-- Base_link-->
     <xacro:base_link name="base_link" parent="base_footprint">
@@ -60,7 +62,26 @@
     </xacro:imu>
         <!--camera-->
-    <xacro:camera name="camera" parent="base_link">
-      <origin rpy="0 0 ${pi} " xyz="-0.465 0 0.284"/>
+    <!-- <xacro:camera name="camera" parent="base_link"  locationprefix="left">
+      <origin rpy="0 0 ${pi} " xyz="-0.405 0.2 0.274"/>
     </xacro:camera>
+    <xacro:camera name="camera" parent="base_link"  locationprefix="right">
+      <origin rpy="0 0 ${pi} " xyz="-0.405 0.2 0.274"/>
+    </xacro:camera> -->
+<!--
+    <xacro:sensor_d435i parent="base_link" use_nominal_extrinsics="$(arg use_nominal_extrinsics)" locationprefix="left">
+      <origin rpy="0 0 ${pi} " xyz="-0.405 0.2 0.274"/>
+    </xacro:sensor_d435i>
+    <xacro:sensor_d435i parent="base_link" use_nominal_extrinsics="$(arg use_nominal_extrinsics)" locationprefix="right">
+      <origin rpy="0 0 ${pi} " xyz="-0.405 -0.2 0.274"/>
+    </xacro:sensor_d435i> -->
+    <!-- Intel Realsense -->
+    <xacro:sensor_intel_d435i prefix="left_realsense" parent="base_link" prefix_topic="left_realsense">
+      <!-- <origin xyz="0.4 0 0.28" rpy="0 0.10 0" /> -->
+      <origin rpy="0 0 ${pi} " xyz="-0.43 -0.2 0.284"/>
+    </xacro:sensor_intel_d435i>
+    <xacro:sensor_intel_d435i prefix="right_realsense" parent="base_link" prefix_topic="right_realsense">
+      <!-- <origin xyz="0.4 0 0.28" rpy="0 0.10 0" /> -->
+      <origin rpy="0 0 ${pi} " xyz="-0.43 0.2 0.284"/>
+    </xacro:sensor_intel_d435i>
     <!--Caster base Hub-->
     <xacro:caster_wheel parent="base_link" locationprefix='back_left' >

File: urdf/amr_mini_xacro.urdf (robot description, URDF)
Before this commit: robot AmrRobot, 18 links, 17 joints
Links:
- removed link camera
- added link left_realsense_base_link
- added link left_realsense_color_frame
- added link left_realsense_color_optical_frame
- added link left_realsense_depth_frame
- added link left_realsense_depth_optical_frame
- added link left_realsense_infra1_frame
- added link left_realsense_infra1_optical_frame
- added link left_realsense_infra2_frame
- added link left_realsense_infra2_optical_frame
- added link left_realsense_link, mass 0.564; collision box size=0.02505 0.09 0.025; visual mesh filename=file:///home/mkutan/Documents/ros2_ws/install/amr_mini_desc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
- added link right_realsense_base_link
- added link right_realsense_color_frame
- added link right_realsense_color_optical_frame
- added link right_realsense_depth_frame
- added link right_realsense_depth_optical_frame
- added link right_realsense_infra1_frame
- added link right_realsense_infra1_optical_frame
- added link right_realsense_infra2_frame
- added link right_realsense_infra2_optical_frame
- added link right_realsense_link, mass 0.564; collision box size=0.02505 0.09 0.025; visual mesh filename=file:///home/mkutan/Documents/ros2_ws/install/amr_mini_desc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
Joints:
- removed joint camera_joint
- added joint left_realsense_base_joint: type fixed, parent base_link, child left_realsense_base_link, origin xyz=-0.43 -0.2 0.284 rpy=0 0 3.141592653589793 
- added joint left_realsense_color_joint: type fixed, parent left_realsense_link, child left_realsense_color_frame, origin xyz=0 0.015 0 rpy=0 0 0
- added joint left_realsense_color_optical_joint: type fixed, parent left_realsense_color_frame, child left_realsense_color_optical_frame, origin xyz=0 0 0 rpy=-1.5707963267948966 0 -1.5707963267948966
- added joint left_realsense_depth_joint: type fixed, parent left_realsense_link, child left_realsense_depth_frame, origin xyz=0 0 0 rpy=0 0 0
- added joint left_realsense_depth_optical_joint: type fixed, parent left_realsense_depth_frame, child left_realsense_depth_optical_frame, origin xyz=0 0 0 rpy=-1.5707963267948966 0 -1.5707963267948966
- added joint left_realsense_infra1_joint: type fixed, parent left_realsense_link, child left_realsense_infra1_frame, origin xyz=0 0.0 0 rpy=0 0 0
- added joint left_realsense_infra1_optical_joint: type fixed, parent left_realsense_infra1_frame, child left_realsense_infra1_optical_frame, origin xyz=0 0 0 rpy=-1.5707963267948966 0 -1.5707963267948966
- added joint left_realsense_infra2_joint: type fixed, parent left_realsense_link, child left_realsense_infra2_frame, origin xyz=0 -0.05 0 rpy=0 0 0
- added joint left_realsense_infra2_optical_joint: type fixed, parent left_realsense_infra2_frame, child left_realsense_infra2_optical_frame, origin xyz=0 0 0 rpy=-1.5707963267948966 0 -1.5707963267948966
- added joint left_realsense_joint: type fixed, parent left_realsense_base_link, child left_realsense_link, origin xyz=-0.01 0.02 0 rpy=0 0 0
- added joint right_realsense_base_joint: type fixed, parent base_link, child right_realsense_base_link, origin xyz=-0.43 0.2 0.284 rpy=0 0 3.141592653589793 
- added joint right_realsense_color_joint: type fixed, parent right_realsense_link, child right_realsense_color_frame, origin xyz=0 0.015 0 rpy=0 0 0
- added joint right_realsense_color_optical_joint: type fixed, parent right_realsense_color_frame, child right_realsense_color_optical_frame, origin xyz=0 0 0 rpy=-1.5707963267948966 0 -1.5707963267948966
- added joint right_realsense_depth_joint: type fixed, parent right_realsense_link, child right_realsense_depth_frame, origin xyz=0 0 0 rpy=0 0 0
- added joint right_realsense_depth_optical_joint: type fixed, parent right_realsense_depth_frame, child right_realsense_depth_optical_frame, origin xyz=0 0 0 rpy=-1.5707963267948966 0 -1.5707963267948966
- added joint right_realsense_infra1_joint: type fixed, parent right_realsense_link, child right_realsense_infra1_frame, origin xyz=0 0.0 0 rpy=0 0 0
- added joint right_realsense_infra1_optical_joint: type fixed, parent right_realsense_infra1_frame, child right_realsense_infra1_optical_frame, origin xyz=0 0 0 rpy=-1.5707963267948966 0 -1.5707963267948966
- added joint right_realsense_infra2_joint: type fixed, parent right_realsense_link, child right_realsense_infra2_frame, origin xyz=0 -0.05 0 rpy=0 0 0
- added joint right_realsense_infra2_optical_joint: type fixed, parent right_realsense_infra2_frame, child right_realsense_infra2_optical_frame, origin xyz=0 0 0 rpy=-1.5707963267948966 0 -1.5707963267948966
- added joint right_realsense_joint: type fixed, parent right_realsense_base_link, child right_realsense_link, origin xyz=-0.01 0.02 0 rpy=0 0 0

File: urdf/urdf_include/camera.xacro (robot description, xacro)
@@ -1,11 +1,13 @@
 <?xml version="1.0"?>
 <robot xmlns:xacro="http://www.ros.org/wiki/xacro" name="AmrRobot">
-    <xacro:macro name="camera" params="name parent *origin">
+    <xacro:arg name="use_nominal_extrinsics" default="false"/>
+    <xacro:include filename="$(find amr_mini_description)/urdf/urdf_include/_d435i.urdf.xacro" />
+    <xacro:macro name="camera" params="name parent *origin locationprefix">
         <joint name="${name}_joint" type="fixed">
             <xacro:insert_block name="origin" />
             <parent link="${parent}" />
-            <child link="${name}" />
+            <child link="${locationprefix}_${name}" />
         </joint>
-        <link name="${name}">
+        <!-- <link name="${name}">
             <visual>
                 <origin xyz="0 0 0" rpy="1.57 0 1.57" />
@@ -24,5 +26,5 @@
                 l="0.05"
                 o_xyz="0 0 0" o_rpy="0 0 0" />
-        </link>
+        </link> -->
        <gazebo reference="${name}">
         <sensor type="depth" name="depth_camera">
@@ -30,5 +32,5 @@
             <update_rate>10.0</update_rate>
             <plugin name="${name}_depth_plugin" filename="libgazebo_ros_camera.so">
-              <ros>
+              <!-- <ros>
                 <namespace>amr_mini_description</namespace>
                 <remapping>custom_camera/image_raw:=custom_camera/custom_image</remapping>
@@ -37,7 +39,7 @@
                 <remapping>custom_camera/camera_info_depth:=custom_camera/custom_info_depth</remapping>
                 <remapping>custom_camera/points:=custom_camera/custom_points</remapping>
-              </ros>
-            <camera_name>custom_camera</camera_name>
-              <frame_name>${name}</frame_name>
+              </ros> -->
+            <camera_name>${locationprefix}_${name}_custom_camera</camera_name>
+              <frame_name>${locationprefix}_${name}</frame_name>
               <hack_baseline>0.07</hack_baseline>
                <min_depth>0.001</min_depth>
@@ -51,11 +53,11 @@
             <update_rate>30.0</update_rate>
             <plugin name="${name}_rqb_plugin" filename="libgazebo_ros_camera.so">
-                <ros>
+                <!-- <ros>
                     <namespace>amr_mini_description</namespace>
                     <remapping>image_raw:=custom_img</remapping>
                     <remapping>camera_info:=custom_info</remapping>
-                  </ros>
-                  <camera_name>rgb_cam</camera_name>
-                  <frame_name>${name}</frame_name>
+                  </ros> -->
+                  <camera_name>${locationprefix}_${name}_rgb_cam</camera_name>
+                  <frame_name>${locationprefix}_${name}</frame_name>
                   <hack_baseline>0.07</hack_baseline>
             </plugin>

Commit message: Amr_mini

File: urdf/amr_mini.xacro (robot description, xacro)
@@ -14,5 +14,4 @@
     <xacro:property name="amr_mini_front_caster_wheel_base_dz" value="0.0536"/>
     <xacro:property name="locationright" value="1"/>
-   <xacro:arg name="use_nominal_extrinsics" default="false"/>
     <!-- include-->
   <xacro:include filename="$(find amr_mini_description)/urdf/urdf_include/base_link.xacro"/>
@@ -23,5 +22,4 @@
   <xacro:include filename="$(find amr_mini_description)/urdf/urdf_include/imu.xacro"/>
   <xacro:include filename="$(find amr_mini_description)/urdf/urdf_include/gazebo.xacro"/>
-  <xacro:include filename="$(find amr_mini_description)/urdf/urdf_include/_d435i.urdf.xacro" />
   <xacro:include filename="$(find amr_mini_description)/urdf/urdf_include/intel_d435.urdf.xacro" />
     <!-- Base_link-->
@@ -53,8 +51,4 @@
       <origin rpy="0 0 -${pi}" xyz="-${lidar_x} -${lidar_y} ${lidar_z}"/>
     </xacro:lidar>
-    <!-- Lidar-->
-    <!-- <xacro:lidar name="main_lidar" parent="base_link">
-      <origin rpy="${pi} 0 0" xyz="0 0  ${lidar_z+0.165}"/>
-    </xacro:lidar> -->
     <!--imu-->
     <xacro:imu name="imu" parent="base_link">
@@ -65,14 +59,5 @@
       <origin rpy="0 0 ${pi} " xyz="-0.405 0.2 0.274"/>
     </xacro:camera>
-    <xacro:camera name="camera" parent="base_link"  locationprefix="right">
-      <origin rpy="0 0 ${pi} " xyz="-0.405 0.2 0.274"/>
-    </xacro:camera> -->
-<!--
-    <xacro:sensor_d435i parent="base_link" use_nominal_extrinsics="$(arg use_nominal_extrinsics)" locationprefix="left">
-      <origin rpy="0 0 ${pi} " xyz="-0.405 0.2 0.274"/>
-    </xacro:sensor_d435i>
-    <xacro:sensor_d435i parent="base_link" use_nominal_extrinsics="$(arg use_nominal_extrinsics)" locationprefix="right">
-      <origin rpy="0 0 ${pi} " xyz="-0.405 -0.2 0.274"/>
-    </xacro:sensor_d435i> -->
+  -->
     <!-- Intel Realsense -->
     <xacro:sensor_intel_d435i prefix="left_realsense" parent="base_link" prefix_topic="left_realsense">

File: urdf/urdf_include/base_link.xacro (robot description, xacro)
@@ -13,10 +13,10 @@
           <origin rpy="${pi} 0 0" xyz="-0.47 0.3255 0.27"/>
             <geometry>
-              <mesh filename="file://$(find amr_mini_description)/AmrMini_models/Amr_mini/meshes/sase.stl" scale="0.001 0.001 0.001"/>
+              <mesh filename="file://$(find amr_mini_description)/meshes/sase.stl" scale="0.001 0.001 0.001"/>
             </geometry>
           </visual>
           <collision>
             <geometry>
-              <mesh filename="file://$(find amr_mini_description)/AmrMini_models/Amr_mini/meshes/sase.stl" scale="0.001 0.001 0.001"/>
+              <mesh filename="file://$(find amr_mini_description)/meshes/sase.stl" scale="0.001 0.001 0.001"/>
             </geometry>
             <origin rpy="${pi} 0 0" xyz="-0.47 0.3255 0.27"/>

File: urdf/urdf_include/camera.xacro (robot description, xacro)
@@ -2,5 +2,4 @@
 <robot xmlns:xacro="http://www.ros.org/wiki/xacro" name="AmrRobot">
     <xacro:arg name="use_nominal_extrinsics" default="false"/>
-    <xacro:include filename="$(find amr_mini_description)/urdf/urdf_include/_d435i.urdf.xacro" />
     <xacro:macro name="camera" params="name parent *origin locationprefix">
         <joint name="${name}_joint" type="fixed">
@@ -13,5 +12,5 @@
                 <origin xyz="0 0 0" rpy="1.57 0 1.57" />
                 <geometry>
-                    <mesh filename="file://$(find amr_mini_description)/AmrMini_models/Amr_mini/meshes/camera.dae" />
+                    <mesh filename="file://$(find amr_mini_description)/meshes/camera.dae" />
                 </geometry>
             </visual>
@@ -19,5 +18,5 @@
                 <origin xyz="0 0 0" rpy="1.57 0 1.57" />
                 <geometry>
-                    <mesh filename="file://$(find amr_mini_description)/AmrMini_models/Amr_mini/meshes/camera.dae" />
+                    <mesh filename="file://$(find amr_mini_description)/meshes/camera.dae" />
                 </geometry>
             </collision>

File: urdf/urdf_include/caster_wheel.xacro (robot description, xacro)
@@ -28,10 +28,10 @@
           <origin rpy="0 0 0" xyz="0 0 0"/>
             <geometry>
-              <mesh filename="file://$(find amr_mini_description)/AmrMini_models/Amr_mini/meshes/caster_wheel_base.stl" scale="1 1 0.9"/>
+              <mesh filename="file://$(find amr_mini_description)/meshes/caster_wheel_base.stl" scale="1 1 0.9"/>
             </geometry>
           </visual>
           <collision>
             <geometry>
-              <mesh filename="file://$(find amr_mini_description)/AmrMini_models/Amr_mini/meshes/caster_wheel_base.stl" scale="1 1 0.9"/>
+              <mesh filename="file://$(find amr_mini_description)/meshes/caster_wheel_base.stl" scale="1 1 0.9"/>
             </geometry>
             <origin rpy="0 0 0" xyz="0 0 0"/>

File: urdf/urdf_include/imu.xacro (robot description, xacro)
@@ -11,5 +11,5 @@
                <origin xyz="0  0 -0.04" rpy="0 0 0" />
                 <geometry>
-                    <mesh filename="file://$(find amr_mini_description)/AmrMini_models/Amr_mini/meshes/imu.stl" scale="0.001 0.001 0.001" />
+                    <mesh filename="file://$(find amr_mini_description)/meshes/imu.stl" scale="0.001 0.001 0.001" />
                 </geometry>
             </visual>
@@ -17,5 +17,5 @@
                 <origin xyz="0  0 -0.04" rpy="0 0 0" />
                 <geometry>
-                    <mesh filename="file://$(find amr_mini_description)/AmrMini_models/Amr_mini/meshes/imu.stl" scale="0.001 0.001 0.001" />
+                    <mesh filename="file://$(find amr_mini_description)/meshes/imu.stl" scale="0.001 0.001 0.001" />
                 </geometry>
             </collision>

File: urdf/urdf_include/intel_d435.urdf.xacro (robot description, xacro)
@@ -45,5 +45,5 @@
         <geometry>
           <!-- <box size="${d435_cam_width} ${d435_cam_height} ${d435_cam_depth}"/> -->
-           <mesh filename="file://$(find amr_mini_description)/AmrMini_models/Amr_mini/meshes/camera.dae" />
+           <mesh filename="file://$(find amr_mini_description)/meshes/camera.dae" />
         </geometry>
       </visual>

File: urdf/urdf_include/lidar.xacro (robot description, xacro)
@@ -13,5 +13,5 @@
           <visual>
               <geometry>
-                <mesh filename="file://$(find amr_mini_description)/AmrMini_models/Amr_mini/meshes/lidar.stl" scale="0.001 0.001 0.001"/>
+                <mesh filename="file://$(find amr_mini_description)/meshes/lidar.stl" scale="0.001 0.001 0.001"/>
               </geometry>
               <origin rpy="${pi} 0 -${pi/1.25}" xyz="-0.075 0.02 0"/>
@@ -19,5 +19,5 @@
             <collision>
               <geometry>
-                <mesh filename="file://$(find amr_mini_description)/AmrMini_models/Amr_mini/meshes/lidar.stl" scale="0.001 0.001 0.001"/>
+                <mesh filename="file://$(find amr_mini_description)/meshes/lidar.stl" scale="0.001 0.001 0.001"/>
               </geometry>
               <origin rpy="${pi} 0 -${pi/1.25}" xyz="-0.078 0 0"/>

File: urdf/urdf_include/motor.xacro (robot description, xacro)
@@ -12,5 +12,5 @@
         <visual>
             <geometry>
-              <mesh filename="file://$(find amr_mini_description)/AmrMini_models/Amr_mini/meshes/motor.stl" scale="0.001 0.001 0.00065"/>
+              <mesh filename="file://$(find amr_mini_description)/meshes/motor.stl" scale="0.001 0.001 0.00065"/>
             </geometry>
             <origin rpy="1.57 0 0 " xyz="0 0.05 0"/>
@@ -18,5 +18,5 @@
           <collision>
             <geometry>
-              <mesh filename="file://$(find amr_mini_description)/AmrMini_models/Amr_mini/meshes/motor.stl" scale="0.001 0.001 0.00065"/>
+              <mesh filename="file://$(find amr_mini_description)/meshes/motor.stl" scale="0.001 0.001 0.00065"/>
             </geometry>
             <origin rpy="1.57 0 0 " xyz="0 0.05 0"/>

File: urdf/urdf_include/wheel.xacro (robot description, xacro)
@@ -18,10 +18,10 @@
                 <origin rpy="${pi/2} 0 ${pi/2.0*(reflect - 1)}" xyz="${reflect*wheel_location_x} ${reflect*wheel_location_y} ${wheel_location_z}"/>
                 <geometry>
-                <mesh filename="file://$(find amr_mini_description)/AmrMini_models/Amr_mini/meshes/wheel.STL" scale="0.001 0.001 0.001"/>
+                <mesh filename="file://$(find amr_mini_description)/meshes/wheel.STL" scale="0.001 0.001 0.001"/>
                 </geometry>
             </visual>
             <collision>
                 <geometry>
-                    <mesh filename="file://$(find amr_mini_description)/AmrMini_models/Amr_mini/meshes/wheel.STL" scale="0.001 0.001 0.001"/>
+                    <mesh filename="file://$(find amr_mini_description)/meshes/wheel.STL" scale="0.001 0.001 0.001"/>
                 </geometry>
                 <origin rpy="${pi/2} 0 ${pi/2.0*(reflect - 1)}" xyz="${reflect*wheel_location_x} ${reflect*wheel_location_y} ${wheel_location_z}"/>
