Commit message: Amr_mini

File: urdf/amr_mini.xacro (robot description, xacro)
@@ -22,4 +22,5 @@
   <xacro:include filename="$(find amr_mini_description)/urdf/urdf_include/imu.xacro"/>
   <xacro:include filename="$(find amr_mini_description)/urdf/urdf_include/gazebo.xacro"/>
+  <!-- <xacro:include filename="$(find amr_mini_description)/urdf/urdf_include/camera.xacro" /> -->
   <xacro:include filename="$(find amr_mini_description)/urdf/urdf_include/intel_d435.urdf.xacro" />
     <!-- Base_link-->
@@ -56,5 +57,5 @@
     </xacro:imu>
         <!--camera-->
-    <!-- <xacro:camera name="camera" parent="base_link"  locationprefix="left">
+    <!-- <xacro:camera name="camera" parent="base_link">
       <origin rpy="0 0 ${pi} " xyz="-0.405 0.2 0.274"/>
     </xacro:camera>
@@ -62,9 +63,7 @@
     <!-- Intel Realsense -->
     <xacro:sensor_intel_d435i prefix="left_realsense" parent="base_link" prefix_topic="left_realsense">
-      <!-- <origin xyz="0.4 0 0.28" rpy="0 0.10 0" /> -->
       <origin rpy="0 0 ${pi} " xyz="-0.43 -0.2 0.284"/>
     </xacro:sensor_intel_d435i>
     <xacro:sensor_intel_d435i prefix="right_realsense" parent="base_link" prefix_topic="right_realsense">
-      <!-- <origin xyz="0.4 0 0.28" rpy="0 0.10 0" /> -->
       <origin rpy="0 0 ${pi} " xyz="-0.43 0.2 0.284"/>
     </xacro:sensor_intel_d435i>

File: urdf/urdf_include/camera.xacro (robot description, xacro)
@@ -1,12 +1,11 @@
 <?xml version="1.0"?>
 <robot xmlns:xacro="http://www.ros.org/wiki/xacro" name="AmrRobot">
-    <xacro:arg name="use_nominal_extrinsics" default="false"/>
-    <xacro:macro name="camera" params="name parent *origin locationprefix">
+    <xacro:macro name="camera" params="name parent *origin">
         <joint name="${name}_joint" type="fixed">
             <xacro:insert_block name="origin" />
             <parent link="${parent}" />
-            <child link="${locationprefix}_${name}" />
+            <child link="${name}" />
         </joint>
-        <!-- <link name="${name}">
+        <link name="${name}">
             <visual>
                 <origin xyz="0 0 0" rpy="1.57 0 1.57" />
@@ -25,5 +24,5 @@
                 l="0.05"
                 o_xyz="0 0 0" o_rpy="0 0 0" />
-        </link> -->
+        </link>
        <gazebo reference="${name}">
         <sensor type="depth" name="depth_camera">
@@ -31,5 +30,5 @@
             <update_rate>10.0</update_rate>
             <plugin name="${name}_depth_plugin" filename="libgazebo_ros_camera.so">
-              <!-- <ros>
+              <ros>
                 <namespace>amr_mini_description</namespace>
                 <remapping>custom_camera/image_raw:=custom_camera/custom_image</remapping>
@@ -38,7 +37,7 @@
                 <remapping>custom_camera/camera_info_depth:=custom_camera/custom_info_depth</remapping>
                 <remapping>custom_camera/points:=custom_camera/custom_points</remapping>
-              </ros> -->
-            <camera_name>${locationprefix}_${name}_custom_camera</camera_name>
-              <frame_name>${locationprefix}_${name}</frame_name>
+              </ros>
+            <camera_name>custom_camera</camera_name>
+              <frame_name>${name}</frame_name>
               <hack_baseline>0.07</hack_baseline>
                <min_depth>0.001</min_depth>
@@ -52,11 +51,11 @@
             <update_rate>30.0</update_rate>
             <plugin name="${name}_rqb_plugin" filename="libgazebo_ros_camera.so">
-                <!-- <ros>
+                <ros>
                     <namespace>amr_mini_description</namespace>
                     <remapping>image_raw:=custom_img</remapping>
                     <remapping>camera_info:=custom_info</remapping>
-                  </ros> -->
-                  <camera_name>${locationprefix}_${name}_rgb_cam</camera_name>
-                  <frame_name>${locationprefix}_${name}</frame_name>
+                  </ros>
+                  <camera_name>rgb_cam</camera_name>
+                  <frame_name>${name}</frame_name>
                   <hack_baseline>0.07</hack_baseline>
             </plugin>
